File: CAN.kicad_sch (KiCad schematic)
At the start: 5 parts

Commit message: schematic: wip, layout: initial test fit
Signed-off-by: Connor Rigby <connorr@hey.com>
Parts:
- gave numbers to parts that had none: 5
Changed lines of the file:
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@@
   (symbol (lib_id "power:+3V3") (at 71.12 45.72 0) (unit 1)
     (in_bom yes) (on_board yes) (fields_autoplaced)
-    (property "Reference" "#PWR?" (id 0) (at 71.12 49.53 0)
+    (property "Reference" "#PWR0504" (id 0) (at 71.12 49.53 0)
       (effects (font (size 1.27 1.27)) hide)
     )
@@
   (symbol (lib_id "BOM:C_0402_100n") (at 71.12 49.53 0) (unit 1)
     (in_bom yes) (on_board yes) (fields_autoplaced)
-    (property "Reference" "C?" (id 0) (at 73.66 48.2662 0)
+    (property "Reference" "C502" (id 0) (at 73.66 48.2662 0)
       (effects (font (size 1.27 1.27)) (justify left))
     )
@@
   (symbol (lib_id "power:GND") (at 71.12 52.07 0) (unit 1)
     (in_bom yes) (on_board yes) (fields_autoplaced)
-    (property "Reference" "#PWR?" (id 0) (at 71.12 58.42 0)
+    (property "Reference" "#PWR0505" (id 0) (at 71.12 58.42 0)
       (effects (font (size 1.27 1.27)) hide)
     )
@@
   (symbol (lib_id "power:+3V3") (at 43.18 67.31 0) (unit 1)
     (in_bom yes) (on_board yes) (fields_autoplaced)
-    (property "Reference" "#PWR?" (id 0) (at 43.18 71.12 0)
+    (property "Reference" "#PWR0501" (id 0) (at 43.18 71.12 0)
       (effects (font (size 1.27 1.27)) hide)
     )
@@
   (symbol (lib_id "BOM:R_0402_10k") (at 62.23 77.47 0) (unit 1)
     (in_bom yes) (on_board yes) (fields_autoplaced)
-    (property "Reference" "R?" (id 0) (at 64.77 76.1999 0)
+    (property "Reference" "R501" (id 0) (at 64.77 76.1999 0)
       (effects (font (size 1.27 1.27)) (justify left))
     )
@@
   (symbol (lib_id "power:GND") (at 81.28 80.01 0) (unit 1)
     (in_bom yes) (on_board yes) (fields_autoplaced)
-    (property "Reference" "#PWR?" (id 0) (at 81.28 86.36 0)
+    (property "Reference" "#PWR0506" (id 0) (at 81.28 86.36 0)
       (effects (font (size 1.27 1.27)) hide)
     )
@@
   (symbol (lib_id "BOM:C_0402_100n") (at 43.18 77.47 0) (unit 1)
     (in_bom yes) (on_board yes) (fields_autoplaced)
-    (property "Reference" "C?" (id 0) (at 45.72 76.2062 0)
+    (property "Reference" "C501" (id 0) (at 45.72 76.2062 0)
       (effects (font (size 1.27 1.27)) (justify left))
     )
@@
   (symbol (lib_id "BOM:R_120_2512") (at 101.6 67.31 0) (unit 1)
     (in_bom yes) (on_board yes) (fields_autoplaced)
-    (property "Reference" "R?" (id 0) (at 104.14 66.6749 0)
+    (property "Reference" "R502" (id 0) (at 104.14 66.6749 0)
       (effects (font (size 1.27 1.27)) (justify left))
     )
@@
   (symbol (lib_id "power:GND") (at 62.23 80.01 0) (unit 1)
     (in_bom yes) (on_board yes) (fields_autoplaced)
-    (property "Reference" "#PWR?" (id 0) (at 62.23 86.36 0)
+    (property "Reference" "#PWR0503" (id 0) (at 62.23 86.36 0)
       (effects (font (size 1.27 1.27)) hide)
     )
@@
   (symbol (lib_id "BOM:U_SIT1044TK{slash}3") (at 81.28 67.31 0) (unit 1)
     (in_bom yes) (on_board yes) (fields_autoplaced)
-    (property "Reference" "U?" (id 0) (at 83.2994 54.61 0)
+    (property "Reference" "U501" (id 0) (at 83.2994 54.61 0)
       (effects (font (size 1.27 1.27)) (justify left))
     )
@@
   (symbol (lib_id "power:GND") (at 43.18 80.01 0) (unit 1)
     (in_bom yes) (on_board yes) (fields_autoplaced)
-    (property "Reference" "#PWR?" (id 0) (at 43.18 86.36 0)
+    (property "Reference" "#PWR0502" (id 0) (at 43.18 86.36 0)
       (effects (font (size 1.27 1.27)) hide)
     )

Commit message: layout: finalize most of the layout
Signed-off-by: Connor Rigby <connorr@hey.com>
Parts:
- removed C501: C_0402_100n, Capacitor_SMD:C_0402_1005Metric, symbol BOM:C_0402_100n
- removed U501: U_SIT1044TK/3, Package_SON:HVSON-8-1EP_3x3mm_P0.65mm_EP1.6x2.4mm, symbol BOM:U_SIT1044TK/3
- added U501: U_TJA1050, Package_SO:SOIC-8_3.9x4.9mm_P1.27mm, symbol BOM:U_TJA1050
Connections:
- net +3V3: now also R501.1, U501.3 (VCC)
- net CAN_H: now also U501.7 (CANH)
- net CAN_L: now also U501.6 (CANL)
- net CAN_RX: now also U501.4 (RXD)
- net CAN_STB: now also R501.2, U501.8 (S); no longer R501.1
- net CAN_TX: now also U501.1 (TXD)
- net GND: now also U501.2 (GND); no longer R501.2
- no-connect marks 0 -> 1
Other:
- moved on the sheet: R501

Commit message: layout: progress
Signed-off-by: Connor Rigby <connorr@hey.com>
Parts:
- C502: LCSC (none) -> C1525; MPN (none) -> CL05B104KO5NNNC
- R501: LCSC (none) -> C25086; MPN (none) -> 0402WGF100KTCE
- R502: value R_120_2512 -> R_120_1206; footprint Resistor_SMD:R_2512_6332Metric -> Resistor_SMD:R_1206_3216Metric; symbol BOM:R_120_2512 -> BOM:R_120_1206; LCSC (none) -> C17909
Other:
- company: (none) -> Connor Rigby
- title: (none) -> GD32 Development Board
Changed lines of the file:
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@@
 (kicad_sch (version 20211123) (generator eeschema)
   (paper "A4")
+  (title_block
+    (title "GD32 Development Board")
+    (date "2023-01-07")
+    (rev "1")
+    (company "Connor Rigby")
+  )
   (junction (at 101.6 64.77) (diameter 0) (color 0 0 0 0)
   )
@@
       (effects (font (size 1.27 1.27)) hide)
     )
-    (property "Datasheet" "~" (id 3) (at 71.12 49.53 0)
+    (property "Datasheet" "https://datasheet.lcsc.com/lcsc/1810191219_Samsung-Electro-Mechanics-CL05B104KO5NNNC_C1525.pdf" (id 3) (at 71.12 49.53 0)
       (effects (font (size 1.27 1.27)) hide)
     )
     (property "Capicatance" "100n" (id 4) (at 73.66 50.8062 0)
       (effects (font (size 1.27 1.27)) (justify left))
+    )
+    (property "LCSC" "C1525" (id 5) (at 71.12 49.53 0)
+      (effects (font (size 1.27 1.27)) hide)
+    )
+    (property "MPN" "CL05B104KO5NNNC" (id 6) (at 71.12 49.53 0)
+      (effects (font (size 1.27 1.27)) hide)
     )
     (pin "1")
@@
       (effects (font (size 1.27 1.27)) (justify left))
     )
+    (property "LCSC" "C25086" (id 5) (at 54.61 68.58 0)
+      (effects (font (size 1.27 1.27)) hide)
+    )
+    (property "MPN" "0402WGF100KTCE" (id 6) (at 54.61 68.58 0)
+      (effects (font (size 1.27 1.27)) hide)
+    )
     (pin "1")
     (pin "2")
@@
     (pin "1")
   )
-  (symbol (lib_id "BOM:R_120_2512") (at 101.6 67.31 0) (unit 1)
-    (in_bom yes) (on_board yes) (fields_autoplaced)
-    (property "Reference" "R502" (id 0) (at 104.14 66.6749 0)
-      (effects (font (size 1.27 1.27)) (justify left))
-    )
-    (property "Value" "R_120_2512" (id 1) (at 102.362 68.326 0)
+  (symbol (lib_id "BOM:R_120_1206") (at 101.6 67.31 0) (unit 1)
+    (in_bom yes) (on_board yes) (fields_autoplaced)
+    (property "Reference" "R502" (id 0) (at 99.06 66.6749 0)
+      (effects (font (size 1.27 1.27)) (justify right))
+    )
+    (property "Value" "R_120_1206" (id 1) (at 102.362 68.326 0)
       (effects (font (size 1.27 1.27)) (justify left) hide)
     )
-    (property "Footprint" "Resistor_SMD:R_2512_6332Metric" (id 2) (at 101.6 67.31 0)
+    (property "Footprint" "Resistor_SMD:R_1206_3216Metric" (id 2) (at 101.6 67.31 0)
       (effects (font (size 1.27 1.27)) hide)
     )
@@
       (effects (font (size 1.27 1.27)) hide)
     )
-    (property "Resistance" "120" (id 4) (at 104.14 69.215 0)
-      (effects (font (size 1 1)) (justify left))
+    (property "Resistance" "120" (id 4) (at 99.06 69.215 0)
+      (effects (font (size 1 1)) (justify right))
     )
     (property "MPN" "RMCF2512FT120R" (id 5) (at 101.6 67.31 0)
@@
       (effects (font (size 1.27 1.27)) hide)
     )
+    (property "LCSC" "C17909" (id 7) (at 101.6 67.31 0)
+      (effects (font (size 1.27 1.27)) hide)
+    )
