File: USB.kicad_sch (KiCad schematic)
At the start: 5 parts

Commit message: schematic: wip, layout: initial test fit
Signed-off-by: Connor Rigby <connorr@hey.com>
Parts:
- gave numbers to parts that had none: 5
Changed lines of the file:
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@@
     (effects (font (size 1.27 1.27)) (justify right))
   )
-  (hierarchical_label "USB_VBUS" (shape bidirectional) (at 148.59 43.18 180)
+  (hierarchical_label "USB_VBUS" (shape output) (at 148.59 43.18 180)
     (effects (font (size 1.27 1.27)) (justify right))
   )
@@
   (symbol (lib_id "power:GND") (at 49.53 64.77 0) (unit 1)
     (in_bom yes) (on_board yes) (fields_autoplaced)
-    (property "Reference" "#PWR?" (id 0) (at 49.53 71.12 0)
+    (property "Reference" "#PWR0602" (id 0) (at 49.53 71.12 0)
       (effects (font (size 1.27 1.27)) hide)
     )
@@
   (symbol (lib_id "power:+3V3") (at 49.53 41.91 0) (unit 1)
     (in_bom yes) (on_board yes) (fields_autoplaced)
-    (property "Reference" "#PWR?" (id 0) (at 49.53 45.72 0)
+    (property "Reference" "#PWR0601" (id 0) (at 49.53 45.72 0)
       (effects (font (size 1.27 1.27)) hide)
     )
@@
   (symbol (lib_id "BOM:U_TS3USB30ERSWR") (at 116.84 58.42 0) (unit 1)
     (in_bom yes) (on_board yes) (fields_autoplaced)
-    (property "Reference" "U?" (id 0) (at 116.84 38.1 0))
+    (property "Reference" "U601" (id 0) (at 116.84 38.1 0))
     (property "Value" "U_TS3USB30ERSWR" (id 1) (at 116.84 40.64 0))
     (property "Footprint" "BOM:QFN40P140X180X55-10N" (id 2) (at 116.84 58.42 0)
@@
   (symbol (lib_id "power:GND") (at 90.17 78.74 0) (unit 1)
     (in_bom yes) (on_board yes) (fields_autoplaced)
-    (property "Reference" "#PWR?" (id 0) (at 90.17 85.09 0)
+    (property "Reference" "#PWR0605" (id 0) (at 90.17 85.09 0)
       (effects (font (size 1.27 1.27)) hide)
     )
@@
   (symbol (lib_id "power:GND") (at 156.21 58.42 0) (unit 1)
     (in_bom yes) (on_board yes) (fields_autoplaced)
-    (property "Reference" "#PWR?" (id 0) (at 156.21 64.77 0)
+    (property "Reference" "#PWR0606" (id 0) (at 156.21 64.77 0)
       (effects (font (size 1.27 1.27)) hide)
     )
@@
   (symbol (lib_id "BOM:C_0402_100n") (at 49.53 62.23 0) (unit 1)
     (in_bom yes) (on_board yes) (fields_autoplaced)
-    (property "Reference" "C?" (id 0) (at 52.07 60.9662 0)
+    (property "Reference" "C601" (id 0) (at 52.07 60.9662 0)
       (effects (font (size 1.27 1.27)) (justify left))
     )
@@
   (symbol (lib_id "power:GND") (at 59.69 64.77 0) (unit 1)
     (in_bom yes) (on_board yes) (fields_autoplaced)
-    (property "Reference" "#PWR?" (id 0) (at 59.69 71.12 0)
+    (property "Reference" "#PWR0603" (id 0) (at 59.69 71.12 0)
       (effects (font (size 1.27 1.27)) hide)
     )
@@
   (symbol (lib_id "BOM:R_0402_10k") (at 68.58 62.23 0) (unit 1)
     (in_bom yes) (on_board yes) (fields_autoplaced)
-    (property "Reference" "R?" (id 0) (at 71.12 60.9599 0)
+    (property "Reference" "R602" (id 0) (at 71.12 60.9599 0)
       (effects (font (size 1.27 1.27)) (justify left))
     )
@@
   (symbol (lib_id "BOM:R_0402_10k") (at 59.69 62.23 0) (unit 1)
     (in_bom yes) (on_board yes) (fields_autoplaced)
-    (property "Reference" "R?" (id 0) (at 62.23 60.9599 0)
+    (property "Reference" "R601" (id 0) (at 62.23 60.9599 0)
       (effects (font (size 1.27 1.27)) (justify left))
     )
@@
   (symbol (lib_id "power:GND") (at 68.58 64.77 0) (unit 1)
     (in_bom yes) (on_board yes) (fields_autoplaced)
-    (property "Reference" "#PWR?" (id 0) (at 68.58 71.12 0)
+    (property "Reference" "#PWR0604" (id 0) (at 68.58 71.12 0)
       (effects (font (size 1.27 1.27)) hide)
     )
@@
   (symbol (lib_id "bom:J_USB_B_Mini") (at 156.21 48.26 0) (mirror y) (unit 1)
     (in_bom yes) (on_board yes)
-    (property "Reference" "J?" (id 0) (at 156.21 38.1 0))
+    (property "Reference" "J601" (id 0) (at 156.21 38.1 0))
     (property "Value" "J_USB_B_Mini" (id 1) (at 161.29 39.37 0)
       (effects (font (size 1.27 1.27)) (justify left) hide)

Commit message: layout: finalize most of the layout
Signed-off-by: Connor Rigby <connorr@hey.com>
Parts:
- removed J601: J_USB_B_Mini, BOM:EDAC_690-005-299-043, symbol bom:J_USB_B_Mini
- added J601: J_USB_B_Mini, BOM:EDAC_690-005-299-043, symbol BOM:J_USB_B_Mini
Connections:
- net D1_M: now also U601.1 (D1+); no longer U601.7 (D1-)
- net D1_P: now also U601.7 (D1-); no longer U601.1 (D1+)
- net D2_M: now also U601.2 (D2+); no longer U601.6 (D2-)
- net D2_P: now also U601.6 (D2-); no longer U601.2 (D2+)
- net GND: now also J601.5 (GND)
- net USB_CON_DM: now also U601.3 (D+), J601.2 (D-); no longer U601.5 (D-)
- net USB_CON_DP: now also U601.5 (D-), J601.3 (D+); no longer U601.3 (D+)
- net USB_VBUS: now also J601.1 (VBUS)
- new net: J601.S1 (Shield), J601.S2 (Shield), J601.S3 (Shield), J601.S4 (Shield)
Other:
- note added: "USB DP and DM are swapped on purpose it seems like the ESD TS3USB chip was not intended to be used with USB B Mini"
Changed lines of the file:
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@@
   (junction (at 49.53 48.26) (diameter 0) (color 0 0 0 0)
   )
-  (no_connect (at 158.75 58.42))
-  (no_connect (at 148.59 53.34))
+  (no_connect (at 180.34 58.42))
+  (no_connect (at 170.18 53.34))
+  (wire (pts (xy 149.86 50.8) (xy 152.4 48.26))
+    (stroke (width 0) (type default) (color 0 0 0 0))
+  )
+  (wire (pts (xy 93.98 63.5) (xy 96.52 60.96))
+    (stroke (width 0) (type default) (color 0 0 0 0))
+  )
   (wire (pts (xy 99.06 53.34) (xy 59.69 53.34))
     (stroke (width 0) (type default) (color 0 0 0 0))
   )
-  (wire (pts (xy 90.17 60.96) (xy 99.06 60.96))
-    (stroke (width 0) (type default) (color 0 0 0 0))
-  )
-  (wire (pts (xy 90.17 63.5) (xy 99.06 63.5))
+  (wire (pts (xy 83.82 60.96) (xy 93.98 60.96))
+    (stroke (width 0) (type default) (color 0 0 0 0))
+  )
+  (wire (pts (xy 93.98 68.58) (xy 96.52 71.12))
+    (stroke (width 0) (type default) (color 0 0 0 0))
+  )
+  (wire (pts (xy 83.82 63.5) (xy 93.98 63.5))
+    (stroke (width 0) (type default) (color 0 0 0 0))
+  )
+  (wire (pts (xy 96.52 68.58) (xy 99.06 68.58))
     (stroke (width 0) (type default) (color 0 0 0 0))
   )
@@
     (stroke (width 0) (type default) (color 0 0 0 0))
   )
-  (wire (pts (xy 134.62 48.26) (xy 148.59 48.26))
+  (wire (pts (xy 152.4 48.26) (xy 170.18 48.26))
+    (stroke (width 0) (type default) (color 0 0 0 0))
+  )
+  (wire (pts (xy 134.62 50.8) (xy 149.86 50.8))
     (stroke (width 0) (type default) (color 0 0 0 0))
   )
@@
     (stroke (width 0) (type default) (color 0 0 0 0))
   )
-  (wire (pts (xy 134.62 50.8) (xy 148.59 50.8))
+  (wire (pts (xy 152.4 50.8) (xy 170.18 50.8))
+    (stroke (width 0) (type default) (color 0 0 0 0))
+  )
+  (wire (pts (xy 134.62 48.26) (xy 149.86 48.26))
+    (stroke (width 0) (type default) (color 0 0 0 0))
+  )
+  (wire (pts (xy 96.52 71.12) (xy 99.06 71.12))
+    (stroke (width 0) (type default) (color 0 0 0 0))
+  )
+  (wire (pts (xy 96.52 60.96) (xy 99.06 60.96))
+    (stroke (width 0) (type default) (color 0 0 0 0))
+  )
+  (wire (pts (xy 93.98 60.96) (xy 96.52 63.5))
     (stroke (width 0) (type default) (color 0 0 0 0))
   )
@@
     (stroke (width 0) (type default) (color 0 0 0 0))
   )
+  (wire (pts (xy 96.52 63.5) (xy 99.06 63.5))
+    (stroke (width 0) (type default) (color 0 0 0 0))
+  )
   (wire (pts (xy 49.53 41.91) (xy 49.53 48.26))
     (stroke (width 0) (type default) (color 0 0 0 0))
   )
-  (wire (pts (xy 90.17 68.58) (xy 99.06 68.58))
+  (wire (pts (xy 149.86 48.26) (xy 152.4 50.8))
+    (stroke (width 0) (type default) (color 0 0 0 0))
+  )
+  (wire (pts (xy 83.82 68.58) (xy 93.98 68.58))
+    (stroke (width 0) (type default) (color 0 0 0 0))
+  )
+  (wire (pts (xy 93.98 71.12) (xy 96.52 68.58))
     (stroke (width 0) (type default) (color 0 0 0 0))
   )
@@
     (stroke (width 0) (type default) (color 0 0 0 0))
   )
-  (wire (pts (xy 90.17 71.12) (xy 99.06 71.12))
+  (wire (pts (xy 83.82 71.12) (xy 93.98 71.12))
     (stroke (width 0) (type default) (color 0 0 0 0))
   )
@@
     (stroke (width 0) (type default) (color 0 0 0 0))
   )
-  (label "USB_CON_DP" (at 148.59 48.26 180)
+  (text "USB DP and DM are swapped on purpose\nit seems like the ESD TS3USB chip was\nnot intended to be used with USB B Mini\n"
+    (at 132.08 60.96 0)
+    (effects (font (size 1.27 1.27)) (justify left bottom))
+  )
+  (label "USB_CON_DP" (at 170.18 48.26 180)
     (effects (font (size 1.27 1.27)) (justify right bottom))
   )
@@
     (effects (font (size 1.27 1.27)) (justify right bottom))
   )
-  (label "USB_CON_DM" (at 148.59 50.8 180)
-    (effects (font (size 1.27 1.27)) (justify right bottom))
-  )
-  (hierarchical_label "D2_P" (shape bidirectional) (at 90.17 68.58 180)
-    (effects (font (size 1.27 1.27)) (justify right))
-  )
-  (hierarchical_label "D1_P" (shape bidirectional) (at 90.17 60.96 180)
-    (effects (font (size 1.27 1.27)) (justify right))
-  )
-  (hierarchical_label "D2_M" (shape bidirectional) (at 90.17 71.12 180)
-    (effects (font (size 1.27 1.27)) (justify right))
-  )
-  (hierarchical_label "USB_VBUS" (shape output) (at 148.59 43.18 180)
-    (effects (font (size 1.27 1.27)) (justify right))
-  )
-  (hierarchical_label "D1_M" (shape bidirectional) (at 90.17 63.5 180)
+  (label "USB_CON_DM" (at 170.18 50.8 180)
+    (effects (font (size 1.27 1.27)) (justify right bottom))
+  )
+  (hierarchical_label "D2_P" (shape bidirectional) (at 83.82 68.58 180)
+    (effects (font (size 1.27 1.27)) (justify right))
+  )
+  (hierarchical_label "D1_P" (shape bidirectional) (at 83.82 60.96 180)
+    (effects (font (size 1.27 1.27)) (justify right))
+  )
+  (hierarchical_label "D2_M" (shape bidirectional) (at 83.82 71.12 180)
+    (effects (font (size 1.27 1.27)) (justify right))
+  )
+  (hierarchical_label "USB_VBUS" (shape output) (at 170.18 43.18 180)
+    (effects (font (size 1.27 1.27)) (justify right))
+  )
+  (hierarchical_label "D1_M" (shape bidirectional) (at 83.82 63.5 180)
     (effects (font (size 1.27 1.27)) (justify right))
   )
@@
     (pin "1")
   )
-  (symbol (lib_id "power:GND") (at 156.21 58.42 0) (unit 1)
-    (in_bom yes) (on_board yes) (fields_autoplaced)
-    (property "Reference" "#PWR0606" (id 0) (at 156.21 64.77 0)
-      (effects (font (size 1.27 1.27)) hide)
-    )
-    (property "Value" "GND" (id 1) (at 156.21 63.5 0))
-    (property "Footprint" "" (id 2) (at 156.21 58.42 0)
-      (effects (font (size 1.27 1.27)) hide)
-    )
-    (property "Datasheet" "" (id 3) (at 156.21 58.42 0)
+  (symbol (lib_id "power:GND") (at 177.8 58.42 0) (unit 1)
+    (in_bom yes) (on_board yes) (fields_autoplaced)
+    (property "Reference" "#PWR0606" (id 0) (at 177.8 64.77 0)
+      (effects (font (size 1.27 1.27)) hide)
+    )
+    (property "Value" "GND" (id 1) (at 177.8 63.5 0))
+    (property "Footprint" "" (id 2) (at 177.8 58.42 0)
+      (effects (font (size 1.27 1.27)) hide)
+    )
+    (property "Datasheet" "" (id 3) (at 177.8 58.42 0)
       (effects (font (size 1.27 1.27)) hide)
     )
@@
     (pin "1")
   )
-  (symbol (lib_id "bom:J_USB_B_Mini") (at 156.21 48.26 0) (mirror y) (unit 1)
-    (in_bom yes) (on_board yes)
-    (property "Reference" "J601" (id 0) (at 156.21 38.1 0))
-    (property "Value" "J_USB_B_Mini" (id 1) (at 161.29 39.37 0)
+  (symbol (lib_id "BOM:J_USB_B_Mini") (at 177.8 48.26 0) (mirror y) (unit 1)
+    (in_bom yes) (on_board yes) (fields_autoplaced)
+    (property "Reference" "J601" (id 0) (at 184.15 48.2599 0)
+      (effects (font (size 1.27 1.27)) (justify right))
+    )
+    (property "Value" "J_USB_B_Mini" (id 1) (at 172.72 39.37 0)
       (effects (font (size 1.27 1.27)) (justify left) hide)
     )
-    (property "Footprint" "BOM:EDAC_690-005-299-043" (id 2) (at 152.4 49.53 0)
-      (effects (font (size 1.27 1.27)) hide)
-    )
-    (property "Datasheet" "http://files.edac.net/edac/content/1/690-005-299-043.pdf" (id 3) (at 152.4 49.53 0)
-      (effects (font (size 1.27 1.27)) hide)
-    )
-    (property "Digikey" "151-1206-1-ND" (id 4) (at 156.21 48.26 0)
-      (effects (font (size 1.27 1.27)) hide)
-    )
-    (property "MPN" "690-005-299-043" (id 5) (at 156.21 48.26 0)
-      (effects (font (size 1.27 1.27)) hide)
-    )
-    (property "LCSC" "C3039330" (id 6) (at 156.21 48.26 0)
-      (effects (font (size 1.27 1.27)) hide)
-    )
+    (property "Footprint" "BOM:EDAC_690-005-299-043" (id 2) (at 181.61 49.53 0)
+      (effects (font (size 1.27 1.27)) hide)
+    )
+    (property "Datasheet" "http://files.edac.net/edac/content/1/690-005-299-043.pdf" (id 3) (at 181.61 49.53 0)
+      (effects (font (size 1.27 1.27)) hide)
+    )
+    (property "Digikey" "151-1206-1-ND" (id 4) (at 177.8 48.26 0)
+      (effects (font (size 1.27 1.27)) hide)
+    )
+    (property "MPN" "690-005-299-043" (id 5) (at 177.8 48.26 0)
+      (effects (font (size 1.27 1.27)) hide)
+    )
+    (property "LCSC" "C3039330" (id 6) (at 177.8 48.26 0)
+      (effects (font (size 1.27 1.27)) hide)
+    )

Commit message: layout: progress
Signed-off-by: Connor Rigby <connorr@hey.com>
Parts:
- added NT601, NT602: NetTie_2, symbol Device:NetTie_2
- C601: LCSC (none) -> C1525; MPN (none) -> CL05B104KO5NNNC
- R601, R602: LCSC (none) -> C25086; MPN (none) -> 0402WGF100KTCE
Connections:
- net +3V3: now also NT601.2; no longer C601.1, U601.9 (VCC)
- net GND: now also NT602.1; no longer U601.4 (GND)
- new net USB_ESD_GND: NT602.2, U601.4 (GND)
- new net USB_ESD_VCC: C601.1, NT601.1, U601.9 (VCC)
Other:
- company: (none) -> Connor Rigby
- title: (none) -> GD32 Development Board
Changed lines of the file:
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@@
 (kicad_sch (version 20211123) (generator eeschema)
   (paper "A4")
+  (title_block
+    (title "GD32 Development Board")
+    (date "2023-01-07")
+    (rev "1")
+    (company "Connor Rigby")
+  )
   (junction (at 49.53 48.26) (diameter 0) (color 0 0 0 0)
   )
   (no_connect (at 180.34 58.42))
   (no_connect (at 170.18 53.34))
+  (wire (pts (xy 82.55 76.2) (xy 99.06 76.2))
+    (stroke (width 0) (type default) (color 0 0 0 0))
+  )
   (wire (pts (xy 149.86 50.8) (xy 152.4 48.26))
     (stroke (width 0) (type default) (color 0 0 0 0))
@@
     (stroke (width 0) (type default) (color 0 0 0 0))
   )
-  (wire (pts (xy 90.17 78.74) (xy 90.17 76.2))
-    (stroke (width 0) (type default) (color 0 0 0 0))
-  )
   (wire (pts (xy 152.4 48.26) (xy 170.18 48.26))
     (stroke (width 0) (type default) (color 0 0 0 0))
@@
     (stroke (width 0) (type default) (color 0 0 0 0))
   )
-  (wire (pts (xy 49.53 41.91) (xy 49.53 48.26))
+  (wire (pts (xy 49.53 35.56) (xy 49.53 43.18))
     (stroke (width 0) (type default) (color 0 0 0 0))
   )
@@
   )
   (wire (pts (xy 93.98 71.12) (xy 96.52 68.58))
-    (stroke (width 0) (type default) (color 0 0 0 0))
-  )
-  (wire (pts (xy 90.17 76.2) (xy 99.06 76.2))
     (stroke (width 0) (type default) (color 0 0 0 0))
   )
@@
     (effects (font (size 1.27 1.27)) (justify right bottom))
   )
+  (label "USB_ESD_VCC" (at 59.69 48.26 0)
+    (effects (font (size 1.27 1.27)) (justify left bottom))
+  )
   (label "DSEL" (at 96.52 58.42 180)
     (effects (font (size 1.27 1.27)) (justify right bottom))
@@
   (label "DSEL" (at 96.52 55.88 180)
     (effects (font (size 1.27 1.27)) (justify right bottom))
+  )
+  (label "USB_ESD_GND" (at 82.55 76.2 0)
+    (effects (font (size 1.27 1.27)) (justify left bottom))
   )
   (label "USB_CON_DM" (at 170.18 50.8 180)
@@
     (pin "1")
   )
-  (symbol (lib_id "power:+3V3") (at 49.53 41.91 0) (unit 1)
-    (in_bom yes) (on_board yes) (fields_autoplaced)
-    (property "Reference" "#PWR0601" (id 0) (at 49.53 45.72 0)
-      (effects (font (size 1.27 1.27)) hide)
-    )
-    (property "Value" "+3V3" (id 1) (at 49.53 36.83 0))
-    (property "Footprint" "" (id 2) (at 49.53 41.91 0)
-      (effects (font (size 1.27 1.27)) hide)
-    )
-    (property "Datasheet" "" (id 3) (at 49.53 41.91 0)
-      (effects (font (size 1.27 1.27)) hide)
-    )
-    (pin "1")
+  (symbol (lib_id "power:+3V3") (at 49.53 35.56 0) (unit 1)
+    (in_bom yes) (on_board yes) (fields_autoplaced)
+    (property "Reference" "#PWR0601" (id 0) (at 49.53 39.37 0)
+      (effects (font (size 1.27 1.27)) hide)
+    )
+    (property "Value" "+3V3" (id 1) (at 49.53 30.48 0))
+    (property "Footprint" "" (id 2) (at 49.53 35.56 0)
+      (effects (font (size 1.27 1.27)) hide)
+    )
+    (property "Datasheet" "" (id 3) (at 49.53 35.56 0)
+      (effects (font (size 1.27 1.27)) hide)
+    )
+    (pin "1")
+  )
+  (symbol (lib_id "Device:NetTie_2") (at 49.53 45.72 90) (unit 1)
+    (in_bom no) (on_board no)
+    (property "Reference" "NT601" (id 0) (at 50.8 44.45 0))
+    (property "Value" "NetTie_2" (id 1) (at 46.99 45.72 0)
+      (effects (font (size 1.27 1.27)) hide)
+    )
+    (property "Footprint" "" (id 2) (at 49.53 45.72 0)
+      (effects (font (size 1.27 1.27)) hide)
+    )
+    (property "Datasheet" "~" (id 3) (at 49.53 45.72 0)
+      (effects (font (size 1.27 1.27)) hide)
+    )
+    (pin "1")
+    (pin "2")
   )
   (symbol (lib_id "BOM:U_TS3USB30ERSWR") (at 116.84 58.42 0) (unit 1)
@@
     (pin "9")
   )
-  (symbol (lib_id "power:GND") (at 90.17 78.74 0) (unit 1)
-    (in_bom yes) (on_board yes) (fields_autoplaced)
-    (property "Reference" "#PWR0605" (id 0) (at 90.17 85.09 0)
-      (effects (font (size 1.27 1.27)) hide)
-    )
-    (property "Value" "GND" (id 1) (at 90.17 83.82 0))
-    (property "Footprint" "" (id 2) (at 90.17 78.74 0)
-      (effects (font (size 1.27 1.27)) hide)
-    )
-    (property "Datasheet" "" (id 3) (at 90.17 78.74 0)
+  (symbol (lib_id "power:GND") (at 77.47 76.2 270) (unit 1)
+    (in_bom yes) (on_board yes) (fields_autoplaced)
+    (property "Reference" "#PWR0605" (id 0) (at 71.12 76.2 0)
+      (effects (font (size 1.27 1.27)) hide)
+    )
+    (property "Value" "GND" (id 1) (at 73.66 76.1999 90)
+      (effects (font (size 1.27 1.27)) (justify right))
+    )
+    (property "Footprint" "" (id 2) (at 77.47 76.2 0)
+      (effects (font (size 1.27 1.27)) hide)
+    )
+    (property "Datasheet" "" (id 3) (at 77.47 76.2 0)
       (effects (font (size 1.27 1.27)) hide)
     )
@@
       (effects (font (size 1.27 1.27)) hide)
     )
-    (property "Datasheet" "~" (id 3) (at 49.53 62.23 0)
+    (property "Datasheet" "https://datasheet.lcsc.com/lcsc/1810191219_Samsung-Electro-Mechanics-CL05B104KO5NNNC_C1525.pdf" (id 3) (at 49.53 62.23 0)
       (effects (font (size 1.27 1.27)) hide)
     )
     (property "Capicatance" "100n" (id 4) (at 52.07 63.5062 0)
       (effects (font (size 1.27 1.27)) (justify left))
+    )
+    (property "LCSC" "C1525" (id 5) (at 49.53 62.23 0)
+      (effects (font (size 1.27 1.27)) hide)
+    )
+    (property "MPN" "CL05B104KO5NNNC" (id 6) (at 49.53 62.23 0)
+      (effects (font (size 1.27 1.27)) hide)
     )
     (pin "1")
@@
       (effects (font (size 1.27 1.27)) (justify left))
     )
+    (property "LCSC" "C25086" (id 5) (at 68.58 62.23 0)
+      (effects (font (size 1.27 1.27)) hide)
+    )
+    (property "MPN" "0402WGF100KTCE" (id 6) (at 68.58 62.23 0)
+      (effects (font (size 1.27 1.27)) hide)
+    )
     (pin "1")
     (pin "2")
@@
       (effects (font (size 1.27 1.27)) (justify left))
     )
+    (property "LCSC" "C25086" (id 5) (at 59.69 62.23 0)
+      (effects (font (size 1.27 1.27)) hide)
+    )
+    (property "MPN" "0402WGF100KTCE" (id 6) (at 59.69 62.23 0)
+      (effects (font (size 1.27 1.27)) hide)
+    )
     (pin "1")
     (pin "2")
@@
     (pin "1")
   )
+  (symbol (lib_id "Device:NetTie_2") (at 80.01 76.2 0) (unit 1)
+    (in_bom no) (on_board no)
+    (property "Reference" "NT602" (id 0) (at 81.28 77.47 0))
+    (property "Value" "NetTie_2" (id 1) (at 80.01 73.66 0)
+      (effects (font (size 1.27 1.27)) hide)
+    )
+    (property "Footprint" "" (id 2) (at 80.01 76.2 0)
+      (effects (font (size 1.27 1.27)) hide)
+    )
+    (property "Datasheet" "~" (id 3) (at 80.01 76.2 0)
+      (effects (font (size 1.27 1.27)) hide)
+    )
+    (pin "1")
+    (pin "2")
+  )
   (symbol (lib_id "BOM:J_USB_B_Mini") (at 177.8 48.26 0) (mirror y) (unit 1)
