File: header1.kicad_sch (KiCad schematic)
At the start: 1 part, among them J801 SPI

Commit message: layout: progress
Signed-off-by: Connor Rigby <connorr@hey.com>
Parts:
- J801: value SPI -> SPI1; now left out of the parts list
Other:
- company: (none) -> Connor Rigby
- title: (none) -> GD32 Development Board
Changed lines of the file:
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@@
 (kicad_sch (version 20211123) (generator eeschema)
   (paper "A4")
+  (title_block
+    (title "GD32 Development Board")
+    (date "2023-01-07")
+    (rev "1")
+    (company "Connor Rigby")
+  )
   (junction (at 73.66 26.67) (diameter 0) (color 0 0 0 0)
   )
@@
   )
   (symbol (lib_id "Connector_Generic:Conn_02x08_Odd_Even") (at 59.69 34.29 0) (mirror x) (unit 1)
-    (in_bom yes) (on_board yes) (fields_autoplaced)
+    (in_bom no) (on_board yes) (fields_autoplaced)
     (property "Reference" "J801" (id 0) (at 60.96 17.78 0))
-    (property "Value" "SPI" (id 1) (at 60.96 20.32 0))
+    (property "Value" "SPI1" (id 1) (at 60.96 20.32 0))
     (property "Footprint" "Connector_PinSocket_2.54mm:PinSocket_2x08_P2.54mm_Horizontal" (id 2) (at 59.69 34.29 0)
       (effects (font (size 1.27 1.27)) hide)
