File: gd32-devboard.kicad_sch (KiCad schematic)
At the start: 0 parts

Commit message: schematic: wip, layout: initial test fit
Signed-off-by: Connor Rigby <connorr@hey.com>
Other:
- sheet Base ports: added BOOST_EN, CAN1_RX, CAN1_TX, CAN_STBY, GPS_PPS, SDIO_CK, SDIO_CMD, SDIO_D0, SDIO_D1, SDIO_D2, SDIO_D3, SPI1_INT, SPI1_IO0, SPI1_IO1, SPI1_MISO, SPI1_MOSI, SPI1_NSS, SPI1_SCK, SPI2_INT, SPI2_MISO, SPI2_MOSI, SPI2_NSS, SPI2_SCK, USART1_RX, USART1_TX, USART2_CTS, USART2_RTS, USART2_RX, USART2_TX, USART3_RX, USART3_TX, USB_DM, USB_DP, USB_VBUS, ~{GPS_RESET}; removed none
- sheet CAN ports: added CAN_H, CAN_L, CAN_RX, CAN_STB, CAN_TX; removed none
- sheet Power ports: added CAN_H, CAN_L, STEP_EN, USB_VBUS, USB_VBUS_ACT; removed none
- sheet Storage ports: added CLK, CMD, DAT0, DAT1, DAT2, DAT3; removed none
- sheet USB ports: added D1_M, D1_P, D2_M, D2_P, DSEL, USB_VBUS; removed none
- sheet Wireless ports: added GPS_PPS, GPS_RX, GPS_TX, HCI_CTS, HCI_EN, HCI_RTS, HCI_RX, HCI_TX, ~{GPS_RESET}; removed none

Commit message: layout: finalize most of the layout
Signed-off-by: Connor Rigby <connorr@hey.com>
Other:
- added sheet Header1 (header1.kicad_sch)
- added sheet Header2 (header2.kicad_sch)

Commit message: layout: progress
Signed-off-by: Connor Rigby <connorr@hey.com>
Other:
- company: (none) -> Connor Rigby
- title: (none) -> GD32 Development Board
