File: base.kicad_sch (KiCad schematic)
At the start: 25 parts

Commit message: schematic: wip, layout: initial test fit
Signed-off-by: Connor Rigby <connorr@hey.com>
Parts:
- added J201: Conn_02x05_Odd_Even, Connector:Tag-Connect_TC2050-IDC-NL_2x05_P1.27mm_Vertical, symbol Connector_Generic:Conn_02x05_Odd_Even
- added J202: J_TC2030-IDC, Connector:Tag-Connect_TC2030-IDC-NL_2x03_P1.27mm_Vertical, symbol bom:J_TC2030-IDC
- FB201: renamed from FB?; footprint (none) -> Inductor_SMD:L_0402_1005Metric
- gave numbers to parts that had none: 24
Connections:
- net GND: now also J201.4 (Pin_4), J201.5 (Pin_5), J201.8 (Pin_8), J201.9 (Pin_9), J202.4 (Pin_4)
- net JTCK: now also J201.7 (Pin_7)
- net JTDI: now also J201.6 (Pin_6)
- net JTDO: now also J201.2 (Pin_2)
- net JTMS: now also J201.3 (Pin_3)
- net USART1_RX: now also J202.3 (Pin_3)
- net USART1_TX: now also J202.5 (Pin_5)
- net ~{RESET}: now also J201.10 (Pin_10)
- net CAN_STBY: now reaches U201.24 (PC4)
- net BOOST_EN: now reaches U201.37 (PC6)
- net GPS_PPS: now reaches U201.38 (PC7)
- net ~{GPS_RESET}: now reaches U201.59 (PB7)
- no-connect marks 0 -> 4
Other:
- note added: "UART"

Commit message: layout: finalize most of the layout
Signed-off-by: Connor Rigby <connorr@hey.com>
Connections:
- net +3.3VA: now also C215.1, FB201.1, U201.13 (VDDA); no longer C216.1, FB201.2
- net +3V3: now also C216.1, FB201.2; no longer C215.1, FB201.1, U201.13 (VDDA)
- net ~{RESET}: no longer J201.10 (Pin_10)
- no-connect marks 4 -> 5
Changed lines of the file:
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@@
   (no_connect (at 187.96 119.38))
   (no_connect (at 213.36 148.59))
+  (no_connect (at 200.66 129.54))
   (no_connect (at 200.66 148.59))
   (no_connect (at 213.36 153.67))
@@
     (stroke (width 0) (type default) (color 0 0 0 0))
   )
+  (wire (pts (xy 158.75 29.21) (xy 158.75 30.48))
+    (stroke (width 0) (type default) (color 0 0 0 0))
+  )
   (wire (pts (xy 95.25 31.75) (xy 95.25 30.48))
     (stroke (width 0) (type default) (color 0 0 0 0))
@@
     (stroke (width 0) (type default) (color 0 0 0 0))
   )
-  (wire (pts (xy 200.66 129.54) (xy 213.36 129.54))
-    (stroke (width 0) (type default) (color 204 102 0 1))
-  )
   (wire (pts (xy 128.27 30.48) (xy 130.81 30.48))
     (stroke (width 0) (type default) (color 0 0 0 0))
@@
     (stroke (width 0) (type default) (color 0 0 0 0))
   )
-  (wire (pts (xy 142.24 29.21) (xy 142.24 30.48))
-    (stroke (width 0) (type default) (color 0 0 0 0))
-  )
   (wire (pts (xy 41.91 130.81) (xy 41.91 134.62))
     (stroke (width 0) (type default) (color 0 0 0 0))
@@
     (stroke (width 0) (type default) (color 0 0 0 0))
   )
-  (wire (pts (xy 158.75 29.21) (xy 158.75 30.48))
+  (wire (pts (xy 142.24 29.21) (xy 142.24 30.48))
     (stroke (width 0) (type default) (color 0 0 0 0))
   )
@@
     (effects (font (size 1.27 1.27)) (justify left bottom))
   )
-  (label "~{RESET}" (at 213.36 129.54 180)
-    (effects (font (size 1.27 1.27)) (justify right bottom))
-  )
   (label "HSI_IN" (at 69.85 88.9 0)
     (effects (font (size 1.27 1.27)) (justify left bottom))
@@
     (pin "1")
   )
+  (symbol (lib_id "power:+3V3") (at 158.75 29.21 0) (unit 1)
+    (in_bom yes) (on_board yes) (fields_autoplaced)
+    (property "Reference" "#PWR0102" (id 0) (at 158.75 33.02 0)
+      (effects (font (size 1.27 1.27)) hide)
+    )
+    (property "Value" "+3V3" (id 1) (at 158.75 24.13 0))
+    (property "Footprint" "" (id 2) (at 158.75 29.21 0)
+      (effects (font (size 1.27 1.27)) hide)
+    )
+    (property "Datasheet" "" (id 3) (at 158.75 29.21 0)
+      (effects (font (size 1.27 1.27)) hide)
+    )
+    (pin "1")
+  )
   (symbol (lib_id "BOM:C_0402_39p") (at 59.69 90.17 0) (unit 1)
     (in_bom yes) (on_board yes) (fields_autoplaced)
@@
     (pin "1")
   )
-  (symbol (lib_id "power:+3.3VA") (at 158.75 29.21 0) (unit 1)
+  (symbol (lib_id "power:+3.3VA") (at 142.24 29.21 0) (unit 1)
     (in_bom yes) (on_board yes) (fields_autoplaced)
-    (property "Reference" "#PWR0227" (id 0) (at 158.75 33.02 0)
+    (property "Reference" "#PWR0227" (id 0) (at 142.24 33.02 0)
       (effects (font (size 1.27 1.27)) hide)
     )
-    (property "Value" "+3.3VA" (id 1) (at 158.75 24.13 0))
-    (property "Footprint" "" (id 2) (at 158.75 29.21 0)
+    (property "Value" "+3.3VA" (id 1) (at 142.24 24.13 0))
+    (property "Footprint" "" (id 2) (at 142.24 29.21 0)
       (effects (font (size 1.27 1.27)) hide)
     )
-    (property "Datasheet" "" (id 3) (at 158.75 29.21 0)
+    (property "Datasheet" "" (id 3) (at 142.24 29.21 0)
       (effects (font (size 1.27 1.27)) hide)
     )
@@
     (pin "2")
   )
-  (symbol (lib_id "power:+3V3") (at 142.24 29.21 0) (unit 1)
-    (in_bom yes) (on_board yes) (fields_autoplaced)
-    (property "Reference" "#PWR0225" (id 0) (at 142.24 33.02 0)
-      (effects (font (size 1.27 1.27)) hide)
-    )
-    (property "Value" "+3V3" (id 1) (at 142.24 24.13 0))
-    (property "Footprint" "" (id 2) (at 142.24 29.21 0)
-      (effects (font (size 1.27 1.27)) hide)
-    )
-    (property "Datasheet" "" (id 3) (at 142.24 29.21 0)
-      (effects (font (size 1.27 1.27)) hide)
-    )
-    (pin "1")
-  )
 )

Commit message: layout: progress
Signed-off-by: Connor Rigby <connorr@hey.com>
Parts:
- C201, C202, C204, C205: LCSC C1563 -> C1562; MPN 0402CG390J500NT -> 0402CG330J500NT
- C203, C208, C209, C211, C212, C213, C214, C215: LCSC (none) -> C1525; MPN (none) -> CL05B104KO5NNNC
- C206, C207: LCSC (none) -> C12530; MPN (none) -> CL05A225MQ5NSNC
- C210: LCSC (none) -> C23733; MPN (none) -> CL05A475MP5NRNC
- C216: LCSC (none) -> C15195; MPN (none) -> CL05B103KB5NNNC
- FB201: value FerriteBead_Small -> FB_0402_1k; symbol BOM:FerriteBead_Small -> BOM:FB_0402_1k; LCSC (none) -> C17909; MPN (none) -> GZ1005U102TF
- J201: now left out of the parts list
- R201, R202, R203: LCSC (none) -> C25086; MPN (none) -> 0402WGF100KTCE
Other:
- company: (none) -> Connor Rigby
- title: (none) -> GD32 Development Board
- moved on the sheet: BT201, C201, C202, C203, C204, C205, C206, C207, C208, C209, C210, C211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

Commit message: production: prepare for fab
Signed-off-by: Connor Rigby <connorr@hey.com>
Parts:
- added D202: LED_YLW, LED_SMD:LED_0603_1608Metric, symbol BOM:LED_YLW
- added D203, D204: LED_GRN, LED_SMD:LED_0603_1608Metric, symbol BOM:LED_GRN
- added R204, R205, R206: R_0603_500, Resistor_SMD:R_0603_1608Metric, symbol BOM:R_0603_500
Connections:
- net +3V3: now also R204.1, R205.1, R206.2
- net LED_STATUS: now reaches U201.57 (PB5)
- net LED_STATUS: now also D204.2 (A)
- net LED_ACT: now reaches U201.8 (PC0)
- net LED_ACT: now also D202.2 (A)
- net LED_LINK: now reaches U201.9 (PC1)
- net LED_LINK: now also D203.2 (A)
- new net LED_ACT_ANODE: D202.1 (K), R204.2
- new net LED_LINK_ANODE: D203.1 (K), R205.2
- new net LED_STATUS_ANODE: D204.1 (K), R206.1

Commit message: release: submit for production
Signed-off-by: Connor Rigby <connorr@hey.com>
Parts:
- FB201: LCSC C17909 -> C19136
Changed lines of the file:
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@@
       (effects (font (size 1.27 1.27)) hide)
     )
-    (property "LCSC" "C17909" (id 5) (at 157.48 43.18 0)
+    (property "LCSC" "C19136" (id 5) (at 157.48 43.18 0)
       (effects (font (size 1.27 1.27)) hide)
     )
