File: gd32-devboard.kicad_pcb (KiCad board)
At the start: 2 copper layers, 50 x 50 mm, 101 parts, among them J201 Conn_02x05_Odd_Even, J202 J_TC2030-IDC, J301 J_TC2030-IDC, J401 DB9_Female_MountingHoles, J601 J_USB_B_Mini, J701 J_Micro_SD_Card, Q301 Q_SOT23_NPN, Q302 Q_SOT23_NPN, U201 U_GD32F405RGT6, U301 U_ATGM336H-5N31, U302 U_ESP32-C3-MINI-1U-N4, U303 U_AT2659, U304 U_RA-01S, U401 U_LM317_TO-252, U402 U_TLV61046ADB, U501 U_SIT1044TK/3, U601 U_TS3USB30ERSWR, Y201 Y_32.768k, Y202 Y_8m

Commit message: layout: finalize most of the layout
Signed-off-by: Connor Rigby <connorr@hey.com>
Parts:
- removed C404, C501: C_0402_100n, Capacitor_SMD:C_0402_1005Metric
- added J801: SPI, Connector_PinSocket_2.54mm:PinSocket_2x08_P2.54mm_Horizontal, F.Cu at (58.3, 71.2)
- added J901: Conn_02x05_Counter_Clockwise, Connector_PinSocket_2.54mm:PinSocket_2x05_P2.54mm_Horizontal, F.Cu at (58.3, 49.6)
- added TP404: GND, TestPoint:TestPoint_Pad_D1.0mm, F.Cu at (37.6, 49.0)
- BT201, BT301: moved to F.Cu
- U301: footprint RF_GPS:ublox_MAX -> BOM:ublox_MAX
- U304: footprint RF_Module:Ai-Thinker-Ra-01-LoRa -> BOM:Ai-Thinker-Ra-01-LoRa
- U501: value U_SIT1044TK/3 -> U_TJA1050; footprint Package_SON:HVSON-8-1EP_3x3mm_P0.65mm_EP1.6x2.4mm -> Package_SO:SOIC-8_3.9x4.9mm_P1.27mm
- moved R308 120.3 mm to (24.1, 101.1), turned to -90 degrees
- moved C303 108.0 mm to (25.8, 86.2)
- moved C307 105.8 mm to (22.9, 106.5)
- moved C305 101.6 mm to (28.2, 105.1)
- moved C301 101.3 mm to (23.1, 86.2)
- moved TP301 99.1 mm to (33.5, 94.6), turned to 180 degrees
- moved C304 96.8 mm to (26.4, 101.1), turned to -90 degrees
- moved Q302 94.1 mm to (40.0, 84.3), turned to 180 degrees
- moved R301 93.8 mm to (39.3, 87.4), turned to -90 degrees
- moved R704 88.0 mm to (34.2, 61.2), turned to -45 degrees
- moved C308 87.9 mm to (65.3, 103.6), turned to -90 degrees
- moved L302 87.5 mm to (25.3, 101.1), turned to -90 degrees
- moved R705 86.4 mm to (35.0, 60.4), turned to -45 degrees
- moved R307 84.6 mm to (22.5, 101.1), turned to -90 degrees
- moved C701 84.0 mm to (26.2, 73.9), turned to -90 degrees
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Connections:
- net Net-(C303-Pad2) renamed /Wireless/GPS_VBACKUP
- C215 pad 1: +3V3 -> +3.3VA
- C216 pad 1: +3.3VA -> +3V3
- C701 pad 2: Net-(C701-Pad2) -> GND
- D404 pad 2: /Power/12VIN -> /Power/VIN
- FB201 pad 1: +3V3 -> +3.3VA
- FB201 pad 2: +3.3VA -> +3V3
- J201 pad 10: /Base/~{RESET} -> unconnected-(J201-Pad10)
- J701 pad 6: Net-(C701-Pad2) -> GND
- L401 pad 1: /Power/SW -> /Power/USB_VBUS
- L401 pad 2: /Power/VOUT -> /Power/SW
- R501 pad 1: /Base/CAN_STBY -> +3V3
- R501 pad 2: GND -> /Base/CAN_STBY
- U201 pad 13: +3V3 -> +3.3VA
- U501 pad 5: +3V3 -> unconnected-(U501-Pad5)
- U601 pad 1: /Base/USB_DP -> /Base/USB_DM
- U601 pad 2: /USB/D2_P -> /USB/D2_M
- U601 pad 3: /USB/USB_CON_DP -> /USB/USB_CON_DM
- U601 pad 5: /USB/USB_CON_DM -> /USB/USB_CON_DP
- U601 pad 6: /USB/D2_M -> /USB/D2_P
- U601 pad 7: /Base/USB_DM -> /Base/USB_DP
Routing:
- net GND: track 0.00 -> 133.8 mm, vias 0 -> 69
- net /Power/USB_VBUS: track 0.00 -> 93.4 mm, vias 0 -> 4
- net /Base/CAN_STBY: track 0.00 -> 92.2 mm, vias 0 -> 4
- net /Base/USB_DM: track 0.00 -> 77.0 mm, vias 0 -> 4
- net +3V3: track 0.00 -> 76.5 mm, vias 0 -> 26
- net /Base/USB_DP: track 0.00 -> 71.3 mm, vias 0 -> 4
- net /Base/USB_VBUS: track 0.00 -> 71.3 mm, vias 0 -> 2
- net /Wireless/IO9: track 0.00 -> 56.8 mm, vias 0 -> 4
- net /Base/USART1_RX: track 0.00 -> 54.5 mm, vias 0 -> 4
- net /Base/USART1_TX: track 0.00 -> 48.9 mm, vias 0 -> 2
- net /Base/~{GPS_RESET}: track 0.00 -> 42.9 mm, vias 0 -> 2
- net /Storage/DAT1: track 0.00 -> 39.1 mm, vias 0 -> 1
- net /Base/CAN1_TX: track 0.00 -> 36.5 mm
- net /Storage/DAT0: track 0.00 -> 36.3 mm, vias 0 -> 1
- net /Base/SPI2_MISO: track 0.00 -> 35.5 mm, vias 0 -> 2
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- added copper zone on F.Cu, net +3V3
- added copper zone on In2.Cu, net +3V3
- added copper zone on In1.Cu, net GND
- added copper zone on F.Cu, net Net-(BT301-Pad1)
Other:
- board size 50 x 50 mm -> 49.8 x 80.1 mm
- copper layers 2 -> 4

Commit message: layout: progress
Signed-off-by: Connor Rigby <connorr@hey.com>
Parts:
- C305: value C_0402_DNP -> C_0402_470p
- FB201: value FerriteBead_Small -> FB_0402_1k
- J801: value SPI -> SPI1
- J901: value Conn_02x05_Counter_Clockwise -> SPI2
- L301: value L_0402_DNP -> L_6n8
- R502: value R_120_2512 -> R_120_1206; footprint Resistor_SMD:R_2512_6332Metric -> Resistor_SMD:R_1206_3216Metric
- moved U303 7.70 mm to (30.6, 104.8)
- moved C307 5.96 mm to (20.1, 101.2), turned to 90 degrees
- moved L301 5.44 mm to (31.3, 107.0), turned to 180 degrees
- moved C305 2.21 mm to (29.3, 107.0), turned to 180 degrees
- moved J601 1.71 mm to (41.7, 103.2)
- moved C304 1.45 mm to (25.1, 101.8), turned to 180 degrees
- moved C206 1.07 mm to (50.7, 72.1)
- moved R308 1.03 mm to (23.1, 100.8), turned to 0 degrees
- moved C212 1.00 mm to (50.0, 71.3)
- moved R307 0.84 mm to (23.1, 101.8), turned to 0 degrees
- moved L302 0.42 mm to (25.1, 100.8), turned to 180 degrees
- moved R309 0.18 mm to (21.6, 101.2)
Connections:
- net /Wireless/RF_IN renamed /Wireless/LNA_RF_IN
- C601 pad 1: +3V3 -> /USB/USB_ESD_VCC
- J901 pad 1: /Base/SPI2_INT -> /Base/SPI2_SCK
- J901 pad 3: /Base/SPI2_SCK -> /Base/SPI2_NSS
- J901 pad 5: /Base/SPI2_NSS -> /Base/SPI2_INT
- J901 pad 7: /Base/SPI2_MISO -> /Base/SPI2_MOSI
- J901 pad 9: /Base/SPI2_MOSI -> /Base/SPI2_MISO
- U601 pad 4: GND -> /USB/USB_ESD_GND
- U601 pad 9: +3V3 -> /USB/USB_ESD_VCC
Routing:
- net /Wireless/VCC_RF: track 0.00 -> 31.0 mm, vias 0 -> 4
- net /Power/12VIN: track 0.00 -> 20.9 mm
- net /Base/SPI2_MISO: track 35.5 -> 48.6 mm
- net /Base/SPI2_MOSI: track 34.6 -> 46.0 mm
- net GND: track 133.8 -> 144.9 mm, vias 69 -> 67
- net /Wireless/~{GPS_RF_SHDN}: track 0.00 -> 9.92 mm
- net /Base/SPI2_INT: track 21.1 -> 30.5 mm
- net /Base/CAN_STBY: track 92.2 -> 84.5 mm
- net Net-(R307-Pad2): track 0.00 -> 7.41 mm
- net /Base/SPI2_NSS: track 23.2 -> 30.3 mm
- net /Base/SPI1_INT: track 27.3 -> 21.3 mm, vias 2 -> 1
- net /Power/VOUT: track 20.8 -> 15.6 mm
- net /Base/SPI2_SCK: track 21.6 -> 25.2 mm
- net /Wireless/GPS_RF_IN: track 0.00 -> 2.91 mm
- net +3V3: track 76.5 -> 73.6 mm, vias 26 -> 29
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- added copper zone on In1.Cu, net +3V3
- added copper zone on F.Cu, net /Power/VOUT
- added copper zone on F.Cu, net Net-(BT201-Pad1)
Other:
- board size 49.8 x 80.1 mm -> 50 x 80.5 mm
- board text added: "3v3"
- board text added: "ESP UART"
- board text added: "ESP32-C3"
- board text added: "GD32F405"
- board text added: "GND"
- board text added: "GPS"
- board text added: "INT"
- board text added: "IO0"
- board text added: "IO1"
- board text added: "IO8"
- board text added: "IO9"
- board text added: "JTAG"
- board text added: "LORA"
- board text added: "MISO"
- board text added: "MOSI"
- board text added: "NSS"
- board text added: "RX"
- board text added: "SCK"
- board text added: "UART"
- board text added: "USB"
- board text added: "VIN VOUT"
- board text added: "https://cone.codes"

Commit message: production: prepare for fab
Signed-off-by: Connor Rigby <connorr@hey.com>
Parts:
- removed C305: C_0402_470p, Capacitor_SMD:C_0402_1005Metric
- removed C307: C_0402_100n, Capacitor_SMD:C_0402_1005Metric
- removed L301: L_6n8, Inductor_SMD:L_0402_1005Metric
- removed R307: R_0402_DNP, Resistor_SMD:R_0402_1005Metric
- removed R309: R_0402_10k, Resistor_SMD:R_0402_1005Metric
- removed U303: U_AT2659, Package_TO_SOT_SMD:SOT-23-6
- added AE301: 20579-001E, BOM:IPEX_20579-001E, F.Cu at (21.2, 105.4)
- added D202: LED_YLW, LED_SMD:LED_0603_1608Metric, F.Cu at (33.0, 85.4)
- added D203: LED_GRN, LED_SMD:LED_0603_1608Metric, F.Cu at (33.0, 87.0)
- added D204: LED_GRN, LED_SMD:LED_0603_1608Metric, F.Cu at (31.9, 47.9)
- added D405: LED_RED, LED_SMD:LED_0603_1608Metric, F.Cu at (33.5, 47.9)
- added R204: R_0603_500, Resistor_SMD:R_0603_1608Metric, F.Cu at (36.1, 85.4)
- added R205: R_0603_500, Resistor_SMD:R_0603_1608Metric, F.Cu at (36.2, 87.0)
- added R206: R_0603_500, Resistor_SMD:R_0603_1608Metric, F.Cu at (27.4, 47.6)
- added R408: R_0603_500, Resistor_SMD:R_0603_1608Metric, F.Cu at (33.5, 51.0)
- added TP405: 12v, TestPoint:TestPoint_Pad_D1.0mm, F.Cu at (35.4, 53.8)
- L302: value L_0402_DNP -> L_4n7
- moved C304 2.13 mm to (27.0, 100.7), turned to 0 degrees
Connections:
- U201 pad 57: unconnected-(U201-Pad57) -> /Base/LED_STATUS
- U201 pad 8: unconnected-(U201-Pad8) -> /Base/LED_ACT
- U201 pad 9: unconnected-(U201-Pad9) -> /Base/LED_LINK
Routing:
- net /Wireless/VCC_RF: track 31.0 -> 2.90 mm, vias 4 -> 0
- net /Base/LED_STATUS: track 0.00 -> 24.6 mm, vias 0 -> 2
- net /Base/LED_LINK: track 0.00 -> 15.4 mm, vias 0 -> 2
- net /Base/LED_ACT: track 0.00 -> 13.6 mm, vias 0 -> 2
- net /Wireless/~{GPS_RF_SHDN}: track 9.92 -> 0.00 mm
- net Net-(R307-Pad2): track 7.41 -> 0.00 mm
- net +3V3: track 73.6 -> 79.7 mm, vias 29 -> 31
- net /Wireless/ACT_ANT_IN: track 1.05 -> 6.49 mm
- net /Base/CAN_STBY: track 84.5 -> 89.0 mm
- net +12V: track 7.12 -> 11.0 mm
- net /Base/LED_STATUS_ANODE: track 0.00 -> 3.88 mm
- net GND: track 144.9 -> 147.6 mm, vias 67 -> 72
- net /Base/VBAT: track 18.7 -> 16.3 mm
- net /Base/LED_LINK_ANODE: track 0.00 -> 1.55 mm
- net /Base/LED_ACT_ANODE: track 0.00 -> 1.53 mm
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- added copper zone on F.Cu, net /Base/VBAT
Other:
- board text added: "12V"
- board text added: "ACT"
- board text added: "LINK"
- board text added: "STAT"
- board text added: "TX"
- board text added: "VIN"
- board text added: "VOUT"
- board text removed: "VIN VOUT"

Commit message: release: submit for production
Signed-off-by: Connor Rigby <connorr@hey.com>
Parts:
- moved J401 1.50 mm to (33.5, 36.8)
Routing:
- net GND: track 147.6 -> 154.0 mm, vias 72 -> 71
- net /CAN/CAN_L: track 17.7 -> 16.3 mm
- net /Power/12VIN: track 20.9 -> 19.9 mm
- net /CAN/CAN_H: track 19.3 -> 18.3 mm
- net /Base/USART2_CTS: track 33.2 -> 34.1 mm
- net /Wireless/PROG_RX: track 23.4 -> 22.5 mm
- net /Wireless/PROG_TX: track 19.3 -> 18.4 mm
Other:
- board size 50 x 80.5 mm -> 50 x 79.5 mm
