File: storage.kicad_sch (KiCad schematic)
At the start: 7 parts

Commit message: schematic: wip, layout: initial test fit
Signed-off-by: Connor Rigby <connorr@hey.com>
Parts:
- gave numbers to parts that had none: 7
Changed lines of the file:
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@@
   (symbol (lib_id "BOM:R_0402_10k") (at 85.09 68.58 0) (unit 1)
     (in_bom yes) (on_board yes) (fields_autoplaced)
-    (property "Reference" "R?" (id 0) (at 87.63 67.3099 0)
+    (property "Reference" "R703" (id 0) (at 87.63 67.3099 0)
       (effects (font (size 1.27 1.27)) (justify left))
     )
@@
   (symbol (lib_id "power:+3V3") (at 80.01 59.69 0) (unit 1)
     (in_bom yes) (on_board yes) (fields_autoplaced)
-    (property "Reference" "#PWR?" (id 0) (at 80.01 63.5 0)
+    (property "Reference" "#PWR0701" (id 0) (at 80.01 63.5 0)
       (effects (font (size 1.27 1.27)) hide)
     )
@@
   (symbol (lib_id "BOM:R_0402_10k") (at 93.98 68.58 0) (unit 1)
     (in_bom yes) (on_board yes) (fields_autoplaced)
-    (property "Reference" "R?" (id 0) (at 96.52 67.3099 0)
+    (property "Reference" "R704" (id 0) (at 96.52 67.3099 0)
       (effects (font (size 1.27 1.27)) (justify left))
     )
@@
   (symbol (lib_id "BOM:C_0402_100n") (at 80.01 83.82 0) (unit 1)
     (in_bom yes) (on_board yes) (fields_autoplaced)
-    (property "Reference" "C?" (id 0) (at 77.47 82.5562 0)
+    (property "Reference" "C701" (id 0) (at 77.47 82.5562 0)
       (effects (font (size 1.27 1.27)) (justify right))
     )
@@
   (symbol (lib_id "BOM:R_0402_10k") (at 62.23 68.58 0) (unit 1)
     (in_bom yes) (on_board yes) (fields_autoplaced)
-    (property "Reference" "R?" (id 0) (at 64.77 67.3099 0)
+    (property "Reference" "R701" (id 0) (at 64.77 67.3099 0)
       (effects (font (size 1.27 1.27)) (justify left))
     )
@@
   (symbol (lib_id "BOM:R_0402_10k") (at 102.87 68.58 0) (unit 1)
     (in_bom yes) (on_board yes) (fields_autoplaced)
-    (property "Reference" "R?" (id 0) (at 105.41 67.3099 0)
+    (property "Reference" "R705" (id 0) (at 105.41 67.3099 0)
       (effects (font (size 1.27 1.27)) (justify left))
     )
@@
   (symbol (lib_id "BOM:R_0402_10k") (at 69.85 68.58 0) (unit 1)
     (in_bom yes) (on_board yes) (fields_autoplaced)
-    (property "Reference" "R?" (id 0) (at 72.39 67.3099 0)
+    (property "Reference" "R702" (id 0) (at 72.39 67.3099 0)
       (effects (font (size 1.27 1.27)) (justify left))
     )
@@
   (symbol (lib_id "BOM:J_Micro_SD_Card") (at 134.62 81.28 0) (unit 1)
     (in_bom yes) (on_board yes) (fields_autoplaced)
-    (property "Reference" "J?" (id 0) (at 156.21 86.3599 0)
+    (property "Reference" "J701" (id 0) (at 156.21 86.3599 0)
       (effects (font (size 1.27 1.27)) (justify left))
     )

Commit message: layout: finalize most of the layout
Signed-off-by: Connor Rigby <connorr@hey.com>
Connections:
- net GND: now reaches C701.2, J701.6 (VSS)
Changed lines of the file:
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@@
   (junction (at 93.98 64.77) (diameter 0) (color 0 0 0 0)
+  )
+  (junction (at 80.01 86.36) (diameter 0) (color 0 0 0 0)
   )
   (junction (at 80.01 81.28) (diameter 0) (color 0 0 0 0)
@@
     (pin "2")
   )
+  (symbol (lib_id "power:GND") (at 80.01 86.36 0) (unit 1)
+    (in_bom yes) (on_board yes) (fields_autoplaced)
+    (property "Reference" "#PWR0103" (id 0) (at 80.01 92.71 0)
+      (effects (font (size 1.27 1.27)) hide)
+    )
+    (property "Value" "GND" (id 1) (at 80.01 91.44 0)
+      (effects (font (size 1.27 1.27)) hide)
+    )
+    (property "Footprint" "" (id 2) (at 80.01 86.36 0)
+      (effects (font (size 1.27 1.27)) hide)
+    )
+    (property "Datasheet" "" (id 3) (at 80.01 86.36 0)
+      (effects (font (size 1.27 1.27)) hide)
+    )
+    (pin "1")
+  )
   (symbol (lib_id "BOM:R_0402_10k") (at 102.87 68.58 0) (unit 1)

Commit message: layout: progress
Signed-off-by: Connor Rigby <connorr@hey.com>
Parts:
- C701: LCSC (none) -> C1525; MPN (none) -> CL05B104KO5NNNC
- R701, R702, R703, R704, R705: LCSC (none) -> C25086; MPN (none) -> 0402WGF100KTCE
Other:
- company: (none) -> Connor Rigby
- title: (none) -> GD32 Development Board
Changed lines of the file:
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@@
 (kicad_sch (version 20211123) (generator eeschema)
   (paper "A4")
+  (title_block
+    (title "GD32 Development Board")
+    (date "2023-01-07")
+    (rev "1")
+    (company "Connor Rigby")
+  )
   (junction (at 85.09 64.77) (diameter 0) (color 0 0 0 0)
   )
@@
     (property "Resistance" "10k" (id 4) (at 87.63 69.8499 0)
       (effects (font (size 1.27 1.27)) (justify left))
+    )
+    (property "LCSC" "C25086" (id 5) (at 85.09 68.58 0)
+      (effects (font (size 1.27 1.27)) hide)
+    )
+    (property "MPN" "0402WGF100KTCE" (id 6) (at 85.09 68.58 0)
+      (effects (font (size 1.27 1.27)) hide)
     )
     (pin "1")
@@
       (effects (font (size 1.27 1.27)) (justify left))
     )
+    (property "LCSC" "C25086" (id 5) (at 93.98 68.58 0)
+      (effects (font (size 1.27 1.27)) hide)
+    )
+    (property "MPN" "0402WGF100KTCE" (id 6) (at 93.98 68.58 0)
+      (effects (font (size 1.27 1.27)) hide)
+    )
     (pin "1")
     (pin "2")
@@
       (effects (font (size 1.27 1.27)) hide)
     )
-    (property "Datasheet" "~" (id 3) (at 80.01 83.82 0)
+    (property "Datasheet" "https://datasheet.lcsc.com/lcsc/1810191219_Samsung-Electro-Mechanics-CL05B104KO5NNNC_C1525.pdf" (id 3) (at 80.01 83.82 0)
       (effects (font (size 1.27 1.27)) hide)
     )
@@
       (effects (font (size 1.27 1.27)) (justify right))
     )
+    (property "LCSC" "C1525" (id 5) (at 80.01 83.82 0)
+      (effects (font (size 1.27 1.27)) hide)
+    )
+    (property "MPN" "CL05B104KO5NNNC" (id 6) (at 80.01 83.82 0)
+      (effects (font (size 1.27 1.27)) hide)
+    )
     (pin "1")
     (pin "2")
@@
       (effects (font (size 1.27 1.27)) (justify left))
     )
+    (property "LCSC" "C25086" (id 5) (at 62.23 68.58 0)
+      (effects (font (size 1.27 1.27)) hide)
+    )
+    (property "MPN" "0402WGF100KTCE" (id 6) (at 62.23 68.58 0)
+      (effects (font (size 1.27 1.27)) hide)
+    )
     (pin "1")
     (pin "2")
@@
       (effects (font (size 1.27 1.27)) (justify left))
     )
+    (property "LCSC" "C25086" (id 5) (at 102.87 68.58 0)
+      (effects (font (size 1.27 1.27)) hide)
+    )
+    (property "MPN" "0402WGF100KTCE" (id 6) (at 102.87 68.58 0)
+      (effects (font (size 1.27 1.27)) hide)
+    )
     (pin "1")
     (pin "2")
@@
       (effects (font (size 1.27 1.27)) (justify left))
     )
-    (pin "1")
+    (property "LCSC" "C25086" (id 5) (at 69.85 68.58 0)
+      (effects (font (size 1.27 1.27)) hide)
+    )
+    (property "MPN" "0402WGF100KTCE" (id 6) (at 69.85 68.58 0)
+      (effects (font (size 1.27 1.27)) hide)
+    )
+    (pin "1")
